Commit message: update

File: src/robot/urdf/arm.urdf (robot description, URDF)
Before this commit: robot improved_robot, 9 links, 8 joints
Links:
- removed link end_effector
- added link needle; visual cylinder length=3 radius=0.05
- added link sphere; visual sphere radius=1
Joints:
- removed joint arm2_to_end_effector
- added joint arm2_to_sphere: type fixed, parent arm2, child sphere, origin xyz=0 0 7.5 rpy=0 0 0
- added joint sphere_to_needle: type fixed, parent sphere, child needle, origin xyz=0 0 1 rpy=0 0 0

Commit message: Update arm.urdf

File: src/robot/urdf/arm.urdf (robot description, URDF)
Before this commit: robot improved_robot, 10 links, 9 joints
Links:
- link arm1: geometry collision cylinder length=6 radius=1; visual cylinder length=6 radius=1
- link arm1b: geometry collision cylinder length=6 radius=1; visual cylinder length=6 radius=1
- link arm2: geometry collision cylinder length=6 radius=1; visual cylinder length=6 radius=1
- link base_link: geometry collision box size=4 4 1; visual box size=4 4 1
- link needle: geometry collision cylinder length=3 radius=0.05; visual cylinder length=3 radius=0.05
- link pivot1: geometry collision cylinder length=2 radius=1; visual cylinder length=2 radius=1
- link pivot1b: geometry collision cylinder length=2 radius=1; visual cylinder length=2 radius=1
- link pivot2: geometry collision cylinder length=2 radius=1; visual cylinder length=2 radius=1
- link rotator1: geometry collision cylinder length=1 radius=2; visual cylinder length=1 radius=2
- link sphere: geometry collision sphere radius=0; visual sphere radius=1

Commit message: Update arm.urdf

File: src/robot/urdf/arm.urdf (robot description, URDF)
Before this commit: robot improved_robot, 10 links, 9 joints
Links:
- link needle: geometry collision cylinder length=-3 radius=0.05; visual cylinder length=-3 radius=0.05

Commit message: update

File: src/robot/urdf/arm.urdf (robot description, URDF)
Before this commit: robot improved_robot, 10 links, 9 joints
Links:
- added link needle_tip; collision sphere radius=0; visual sphere radius=0.01
- link needle: geometry collision cylinder length=3 radius=0.05; visual cylinder length=3 radius=0.05
Joints:
- added joint needle_to_needle_tip: type fixed, parent needle, child needle_tip, origin xyz=0 0 1.5 rpy=0 0 0

Commit message: Update arm.urdf

File: src/robot/urdf/arm.urdf (robot description, URDF)
Before this commit: robot improved_robot, 11 links, 10 joints
Links:
- link needle_tip: geometry collision sphere radius=0.1; visual sphere radius=0.1

Commit message: Update arm.urdf

File: src/robot/urdf/arm.urdf (robot description, URDF)
Before this commit: robot improved_robot, 11 links, 10 joints
Joints:
- joint needle_to_needle_tip: origin xyz=0 0 1.5 rpy=0 0 0 -> xyz=0 0 2.5 rpy=0 0 0

Commit message: Update arm.urdf

File: src/robot/urdf/arm.urdf (robot description, URDF)
Before this commit: robot improved_robot, 11 links, 10 joints
Links:
- link arm1: geometry collision cylinder length=5.5 radius=0.5; visual cylinder length=5.5 radius=0.5
- link arm1b: geometry collision cylinder length=5.5 radius=0.5; visual cylinder length=5.5 radius=0.5
- link arm2: geometry collision cylinder length=6 radius=0.5; visual cylinder length=6 radius=0.5
- link sphere: geometry collision sphere radius=0.5; visual sphere radius=0.5

Commit message: Update arm.urdf

File: src/robot/urdf/arm.urdf (robot description, URDF)
Before this commit: robot improved_robot, 11 links, 10 joints
Links:
- removed link needle_tip
- link arm2: geometry collision cylinder length=3 radius=0.5; visual cylinder length=3 radius=0.5
- link needle: geometry collision cylinder length=0 radius=0; visual cylinder length=3 radius=0.05
- link pivot1: geometry collision cylinder length=1 radius=0.5; visual cylinder length=1 radius=0.5
- link pivot1b: geometry collision cylinder length=1 radius=0.5; visual cylinder length=1 radius=0.5
- link pivot2: geometry collision cylinder length=1 radius=0.5; visual cylinder length=1 radius=0.5
- link sphere: geometry collision sphere radius=0; visual sphere radius=0.5
Joints:
- removed joint needle_to_needle_tip
- joint arm2_to_sphere: origin xyz=0 0 7.5 rpy=0 0 0 -> xyz=0 0 4.5 rpy=0 0 0

Commit message: Update arm.urdf

File: src/robot/urdf/arm.urdf (robot description, URDF)
Before this commit: robot improved_robot, 10 links, 9 joints
Links:
- link needle: geometry visual cylinder length=3 radius=0.05
- link pivot1: geometry collision cylinder length=1 radius=1; visual cylinder length=1 radius=1
- link pivot1b: geometry collision cylinder length=1 radius=1; visual cylinder length=1 radius=1
- link pivot2: geometry collision cylinder length=1 radius=1; visual cylinder length=1 radius=1
Joints:
- joint sphere_to_needle: axis (none) -> 0 0 1; limit (none) -> lower=0 upper=2 effort=10 velocity=1; origin xyz=0 0 1 rpy=0 0 0 -> xyz=0 0 0 rpy=0 0 0; type fixed -> prismatic

Commit message: Update arm.urdf

File: src/robot/urdf/arm.urdf (robot description, URDF)
Before this commit: robot improved_robot, 10 links, 9 joints
Links:
- link needle: geometry collision cylinder length=0 radius=0; visual cylinder length=3 radius=0.05
Joints:
- joint sphere_to_needle: limit lower=0 upper=2 effort=10 velocity=1 -> lower=-1 upper=2 effort=10 velocity=1

Commit message: Update arm.urdf

File: src/robot/urdf/arm.urdf (robot description, URDF)
Before this commit: robot improved_robot, 10 links, 9 joints
Links:
- link needle: geometry collision cylinder length=0 radius=0; visual cylinder length=1.5 radius=0.05
- link pivot1: geometry collision cylinder length=0.1 radius=0.1; visual cylinder length=1 radius=1
- link pivot1b: geometry collision cylinder length=0.1 radius=0.1; visual cylinder length=1 radius=1
- link pivot2: geometry collision cylinder length=0.1 radius=0.1; visual cylinder length=1 radius=1
Joints:
- joint sphere_to_needle: limit lower=-1 upper=2 effort=10 velocity=1 -> lower=-1.2 upper=0 effort=10 velocity=1; origin xyz=0 0 0 rpy=0 0 0 -> xyz=0 0 1.2 rpy=0 0 0

Commit message: Update arm.urdf

File: src/robot/urdf/arm.urdf (robot description, URDF)
Before this commit: robot robot_arm, 10 links, 9 joints
Links:
- link needle: geometry collision cylinder length=0 radius=0; visual cylinder length=2 radius=0.05
- link sphere: geometry collision sphere radius=0; visual sphere radius=1
Joints:
- joint sphere_to_needle: limit lower=-1.2 upper=0 effort=10 velocity=1 -> lower=0 upper=1 effort=10 velocity=1; origin xyz=0 0 1.2 rpy=0 0 0 -> xyz=0 0 0 rpy=0 0 0

Commit message: Update arm.urdf

File: src/robot/urdf/arm.urdf (robot description, URDF)
Before this commit: robot robot_arm, 10 links, 9 joints
Links:
- link needle: geometry collision cylinder length=2 radius=0.05; visual cylinder length=2 radius=0.05

Commit message: Update arm.urdf

File: src/robot/urdf/arm.urdf (robot description, URDF)
Before this commit: robot robot_arm, 10 links, 9 joints
Links:
- link sphere: geometry collision sphere radius=0; visual sphere radius=0.7

Commit message: update

File: src/robot/urdf/arm.urdf (robot description, URDF)
Before this commit: robot robot_arm, 10 links, 9 joints
Links:
- link sphere: geometry collision sphere radius=0; visual sphere radius=0.5

Commit message: update

File: src/robot/urdf/arm.urdf (robot description, URDF)
Before this commit: robot robot_arm, 10 links, 9 joints
Links:
- link sphere: geometry collision sphere radius=0; visual sphere radius=0.6

Commit message: Update arm.urdf

File: src/robot/urdf/arm.urdf (robot description, URDF)
Before this commit: robot robot_arm, 10 links, 9 joints
Links:
- link needle: geometry collision cylinder length=4 radius=0.05; visual cylinder length=4 radius=0.05
Joints:
- joint sphere_to_needle: limit lower=0 upper=1 effort=10 velocity=1 -> lower=0 upper=4 effort=10 velocity=1

Commit message: Update arm.urdf

File: src/robot/urdf/arm.urdf (robot description, URDF)
Before this commit: robot robot_arm, 10 links, 9 joints
Links:
- link needle: geometry collision cylinder length=0 radius=0; visual cylinder length=4 radius=0.05
