Commit message: all

File: src/robot_moveit/config/gazebo_robot_arm.urdf (robot description, URDF)
Before this commit: robot robot_arm, 10 links, 9 joints
Links:
- link needle: geometry collision cylinder length=0 radius=0; visual cylinder length=4 radius=0.05
- link sphere: geometry collision sphere radius=0; visual sphere radius=0.6
Joints:
- joint sphere_to_needle: limit lower=0 upper=1 effort=10 velocity=1 -> lower=0 upper=4 effort=10 velocity=1
